File: scanner_schematic/scanner_schematic.kicad_sch (KiCad schematic)
At the start: 5 parts, among them M1 Motor_Servo, M2 Motor_Servo, U1 Infrared_Scanner

Commit message: grammar fixes
Parts:
- removed M1: Motor_Servo, symbol Motor:Motor_Servo
Changed lines of the file:
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@@
   (junction (at 124.46 50.8) (diameter 0) (color 0 0 0 0)
-  )
-  (junction (at 102.87 85.09) (diameter 0) (color 0 0 0 0)
   )
   (junction (at 151.13 72.39) (diameter 0) (color 0 0 0 0)
@@
     (stroke (width 0) (type default) (color 0 0 0 0))
   )
-  (wire (pts (xy 101.6 87.63) (xy 101.6 90.17))
-    (stroke (width 0) (type default) (color 0 0 0 0))
-  )
-  (wire (pts (xy 99.06 78.74) (xy 99.06 82.55))
-    (stroke (width 0) (type default) (color 0 0 0 0))
-  )
   (wire (pts (xy 151.13 72.39) (xy 151.13 50.8))
     (stroke (width 0) (type default) (color 0 0 0 0))
   )
-  (wire (pts (xy 101.6 90.17) (xy 106.68 90.17))
-    (stroke (width 0) (type default) (color 0 0 0 0))
-  )
   (wire (pts (xy 104.14 95.25) (xy 106.68 95.25))
     (stroke (width 0) (type default) (color 0 0 0 0))
@@
     (stroke (width 0) (type default) (color 0 0 0 0))
   )
-  (wire (pts (xy 99.06 87.63) (xy 101.6 87.63))
-    (stroke (width 0) (type default) (color 0 0 0 0))
-  )
   (wire (pts (xy 158.75 72.39) (xy 158.75 114.3))
     (stroke (width 0) (type default) (color 0 0 0 0))
@@
     (stroke (width 0) (type default) (color 0 0 0 0))
   )
-  (wire (pts (xy 102.87 85.09) (xy 102.87 101.6))
-    (stroke (width 0) (type default) (color 0 0 0 0))
-  )
   (wire (pts (xy 99.06 101.6) (xy 102.87 101.6))
     (stroke (width 0) (type default) (color 0 0 0 0))
   )
-  (wire (pts (xy 99.06 85.09) (xy 102.87 85.09))
-    (stroke (width 0) (type default) (color 0 0 0 0))
-  )
   (wire (pts (xy 132.08 82.55) (xy 135.89 82.55))
     (stroke (width 0) (type default) (color 0 0 0 0))
@@
     (stroke (width 0) (type default) (color 0 0 0 0))
   )
-  (wire (pts (xy 102.87 85.09) (xy 102.87 50.8))
+  (wire (pts (xy 102.87 50.8) (xy 102.87 101.6))
     (stroke (width 0) (type default) (color 0 0 0 0))
   )
@@
     (pin "9")
   )
-  (symbol (lib_id "Motor:Motor_Servo") (at 91.44 85.09 180) (unit 1)
-    (in_bom yes) (on_board yes) (fields_autoplaced)
-    (property "Reference" "M1" (id 0) (at 90.1811 76.2 0))
-    (property "Value" "Motor_Servo" (id 1) (at 90.1811 78.74 0))
-    (property "Footprint" "" (id 2) (at 91.44 80.264 0)
-      (effects (font (size 1.27 1.27)) hide)
-    )
-    (property "Datasheet" "http://forums.parallax.com/uploads/attachments/46831/74481.png" (id 3) (at 91.44 80.264 0)
-      (effects (font (size 1.27 1.27)) hide)
-    )
-    (pin "1")
-    (pin "2")
-    (pin "3")
-  )
   (symbol (lib_id "Device:C") (at 154.94 72.39 270) (mirror x) (unit 1)
     (in_bom yes) (on_board yes) (fields_autoplaced)
@@
     (pin "2")
   )
-  (symbol (lib_id "power:GND") (at 99.06 78.74 180) (unit 1)
-    (in_bom yes) (on_board yes)
-    (property "Reference" "#PWR0102" (id 0) (at 99.06 72.39 0)
-      (effects (font (size 1.27 1.27)) hide)
-    )
-    (property "Value" "GND" (id 1) (at 99.06 74.93 0))
-    (property "Footprint" "" (id 2) (at 99.06 78.74 0)
-      (effects (font (size 1.27 1.27)) hide)
-    )
-    (property "Datasheet" "" (id 3) (at 99.06 78.74 0)
-      (effects (font (size 1.27 1.27)) hide)
-    )
-    (pin "1")
-  )
   (symbol (lib_id "3d_scanner:infrared_scanner") (at 143.51 78.74 0) (mirror y) (unit 1)
     (in_bom yes) (on_board yes)
@@
       (reference "#PWR0101") (unit 1) (value "GND") (footprint "")
     )
-    (path "/aa6c2633-e6f0-42ba-8d23-56c61505ec84"
-      (reference "#PWR0102") (unit 1) (value "GND") (footprint "")
-    )
     (path "/0cccbd7c-6168-45c6-8aba-93e5a6cab721"
       (reference "#PWR?") (unit 1) (value "+5V") (footprint "")
@@
       (reference "C1") (unit 1) (value "10UF") (footprint "")
     )
-    (path "/33d5138a-15b3-44f6-a8b7-d45e13bbef6b"
-      (reference "M1") (unit 1) (value "Motor_Servo") (footprint "")
-    )
     (path "/1626d76c-560b-4a28-bfa6-3da65b397f13"
